File: Hardware/Boost.brd (EAGLE design)
At the start: 22.9 x 31.8 mm, 42 parts, among them J1 AMP FCI 10103594-0001LF, J2 PTH, J3 PTH, J4 JST, J7 PTH, U1 MCP73831

Commit message: Not sure why this wasn't pushed
Parts:
- removed C10, C9: 4.7uF, SparkFun-Capacitors:0603
- removed D1, D2: 3A/40V/500mV, SparkFun-DiscreteSemi:SMA-DIODE
- removed D4: BLUE, SparkFun-LED:LED-0603
- removed J1: AMP FCI 10103594-0001LF, SparkFun-Connectors:USB-MICROB-PTH
- removed J2: PTH, SparkFun-Connectors:1X02
- removed J4: JST, SparkFun-Connectors:JST-2-SMD
- removed JP5, JP8: STAND-OFF, SparkFun:STAND-OFF
- removed R2: Rprog, SparkFun-Resistors:0805
- removed R5: 2.0k, SparkFun-Resistors:0603
- removed R9: 470, SparkFun-Resistors:0603
- removed S2: (no value), SparkFun-Switches:SWITCH_DPDT_SMD_AYZ0202
- removed SJ3: JUMPER-PAD-3-2OF3_NC_BY_TRACE_SMALL, SparkFun-Passives:PAD-JUMPER-3-2OF3_NC_BY_TRACE_YES_SILK_FULL_BOX
- removed U$2: REVISION, SparkFun-Aesthetics:REVISION
- removed U1: MCP73831, SparkFun-IC-Power:SOT23-5
- J3, J5, J7: device SparkFun-Connectors:1X02 -> SparkFun-Connectors:1X02_NO_SILK
- R3: value 100k -> DNP
- moved U$1 28.4 mm to (6.35, 2.54)
- moved JP7 27.7 mm to (10.2, 2.54)
- moved JP1 20.3 mm to (9.53, 19.1), turned to 270 degrees
- moved J3 19.0 mm to (1.27, 8.89), turned to 270 degrees
- moved C3 17.8 mm to (2.54, 17.1), turned to 270 degrees
- moved JP6 17.8 mm to (2.54, 2.54)
- moved JP2 17.5 mm to (4.83, 0.89)
- moved R6 14.0 mm to (4.45, 13.1), turned to 270 degrees
- moved D3 12.8 mm to (3.94, 6.86), turned to 90 degrees
- moved L1 12.7 mm to (6.35, 17.4)
- moved J7 12.7 mm to (1.27, 11.4), turned to 90 degrees
- moved JP3 11.9 mm to (10.5, 10.4), turned to 45 degrees
- moved J6 11.4 mm to (11.4, 19.1)
- moved C1 11.3 mm to (7.24, 6.60)
- moved C2 11.2 mm to (9.14, 7.11)
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Connections:
- removed net 5VIN: C9.1, D4.A, J1.VBUS, J2.1, U1.4
- removed net N$11: SJ3.2, U1.5
- removed net N$14: R9.1, U1.1
- removed net N$3: R5.1, SJ3.3
- removed net N$5: R2.1, SJ3.1
- removed net N$8: D4.C, R9.2
- removed net SHIELD: J1.P$1, J1.P$10, J1.P$12, J1.P$2, J1.P$3, J1.P$4, J1.P$6, J1.P$8, J1.SHEILD2, J1.SHIELD, J1.SHIELD3, J1.SHIELD4
- net GND: no longer C10.2, C9.2, D1.A, D2.A, J1.GND, J2.2, J4.1, R2.2, R5.2, U1.2
- net N$9: no longer J4.2, S2.1, S2.4
- net VBATT: no longer C10.1, S2.2, S2.5, U1.3
- net VCC: no longer D1.C, D2.C
Routing:
- net N$9: track 33.3 -> 5.08 mm
- net EN: track 2.38 -> 13.3 mm, vias 1 -> 2
- net N$2: track 0.00 -> 5.13 mm
- net N$1: track 0.00 -> 4.21 mm, vias 0 -> 1
- net VCC: track 10.2 -> 13.7 mm, vias 0 -> 1
- net VBATT: track 28.3 -> 25.1 mm, vias 0 -> 1
- net GND: track 2.98 -> 0.00 mm, vias 14 -> 5
- net 5VIN: track 2.52 -> 0.00 mm
- removed copper zone on layer 1, net SHIELD
- removed copper zone on layer 16, net SHIELD
Other:
- board size 22.9 x 31.8 mm -> 12.7 x 20.3 mm
- board text added: "ENB"
- board text added: "Open for 3.3v out"
- board text added: "SWITCH"
- board text added: "VIN"
- board text added: "VOUT"
- board text added: "input: 0.9V to 4.75V"
- board text added: "vX2"
- board text removed: "CHG RATE"
- board text removed: "Charge Boost"
- board text removed: "EN"
- board text removed: "PS"
- board text removed: "PWR"
- board text removed: "STAT"
- board text removed: "VBATT"
- board text removed: "vX1"
