File: Hardware/Boost.sch (EAGLE design)
At the start: 42 parts, among them J1 AMP FCI 10103594-0001LF, J2 PTH, J3 PTH, J4 JST, J7 PTH, U1 MCP73831

Commit message: Not sure why this wasn't pushed
Parts:
- removed C10, C9: 4.7uF, SparkFun-Capacitors:4.7UF0603
- removed D1, D2: 3A/40V/500mV, SparkFun-DiscreteSemi:DIODE-SCHOTTKY-B340A
- removed D4: BLUE, SparkFun-LED:LED-BLUE0603
- removed J1: AMP FCI 10103594-0001LF, SparkFun-Connectors:USB_MICRO-B_HALF_PTH
- removed J2: PTH, SparkFun-Connectors:CONN_02
- removed J4: JST, SparkFun-Connectors:CONN_02-JST-2MM-SMT
- removed JP5, JP8: STAND-OFF, SparkFun:STAND-OFF
- removed R2: Rprog, SparkFun-Resistors:0.75OHM-0805-1/4W-1%
- removed R5: 2.0k, SparkFun-Resistors:2.0KOHM-0603-1/10W-5%
- removed R9: 470, SparkFun-Resistors:470OHM-0603-1/10W-1%
- removed S2: (no value), SparkFun-Switches:SWITCH-DPDT-SMD-AYZ0202
- removed SJ3: JUMPER-PAD-3-2OF3_NC_BY_TRACE_SMALL, SparkFun-Passives:JUMPER-PAD-3-2OF3_NC_BY_TRACE_SMALL
- removed U$2: REVISION, SparkFun-Aesthetics:REVISION
- removed U1: MCP73831, SparkFun-IC-Power:MCP73831
- J3, J5, J7: device SparkFun-Connectors:CONN_02 -> SparkFun-Connectors:CONN_021X02_NO_SILK
- R3: value 100k -> DNP
Connections:
- removed net 5VIN: C9.1, D4.A, J1.VBUS, J2.1, U1.VIN
- removed net N$11: SJ3.2, U1.PROG
- removed net N$14: R9.1, U1.STAT
- removed net N$3: R5.1, SJ3.3
- removed net N$5: R2.1, SJ3.1
- removed net N$8: D4.C, R9.2
- removed net SHIELD: J1.SHIELD
- net GND: no longer C10.2, C9.2, D1.A, D2.A, J1.GND, J2.2, J4.2, R2.2, R5.2, U1.VSS
- net N$9: no longer J4.1, S2.1, S2.4
- net VBATT: no longer C10.1, S2.2, S2.5, U1.VBAT
- net VCC: no longer D1.C, D2.C
Other:
- note added: "Install 100k resistor for inductor current limit"
- note added: "vX2"
- note removed: "500mA"
- note removed: "Aaron Weiss/Patrick Alberts/Toni Klopfenstein"
- note removed: "DNP"
- note removed: "DNP R3: leaving pad in case adjustments are needed for the inductor on prototype"
- note removed: "Ireg = 1000V/Rprog"
- note removed: "LiPo Charger"
- note removed: "SJ3 selects between default 500mA charging rate and user defined charging rate. Rate is defined by value of R10, populated by user."
- note removed: "Switch Bypass"
- note removed: "vX1"
- moved on the sheet: C1, C2, C3, D3, J3, J5, J6, J7, JP1, JP4, L1, R1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
