File: Hardware/ChargeBoost.brd (EAGLE design)
At the start: 20.3 x 31.8 mm, 38 parts, among them J1 AMP FCI 10103594-0001LF, J2 PTH, J3 PTH, J4 JST, J7 PTH, U1 MCP73831

Commit message: Not sure why this wasn't pushed
Parts:
- removed U$2: REVISION, SparkFun-Aesthetics:REVISION
- added TP1: TEST-POINT3, SparkFun-Connectors:PAD.03X.03
- moved J1 0.13 mm to (2.79, 9.53)
Connections:
- net N$14: now also TP1.P$1
