File: Hardware/ChargeBoost.sch (EAGLE design)
At the start: 38 parts, among them J1 AMP FCI 10103594-0001LF, J2 PTH, J3 PTH, J4 JST, J7 PTH, U1 MCP73831

Commit message: Not sure why this wasn't pushed
Parts:
- removed U$2: REVISION, SparkFun-Aesthetics:REVISION
- added TP1: TEST-POINT3, SparkFun-Connectors:TEST-POINT3
Connections:
- net N$14: now also TP1.1
Other:
- note removed: "Aaron Weiss/Patrick Alberts/Toni Klopfenstein"
Changed lines of the file:
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@@
 <part name="U$1" library="SparkFun" deviceset="OSHW-LOGO" device="S"/>
 <part name="JP16" library="SparkFun-Aesthetics" deviceset="FIDUCIAL" device="1X2"/>
-<part name="U$2" library="SparkFun-Aesthetics" deviceset="REVISION" device=""/>
 <part name="GND1" library="SparkFun-PowerSymbols" deviceset="GND" device=""/>
 <part name="LOGO1" library="SparkFun-Aesthetics" deviceset="SFE_LOGO_FLAME" device=".1_INCH"/>
@@
 <part name="JP4" library="SparkFun-Jumpers" deviceset="JUMPER-SMT_2_NO" device="_SILK"/>
 <part name="J7" library="SparkFun-Connectors" deviceset="CONN_02" device="" value="PTH"/>
+<part name="TP1" library="SparkFun-Connectors" deviceset="TEST-POINT" device="3"/>
 </parts>
 <sheets>
@@
 <text x="5.08" y="175.26" size="3.81" layer="97" font="vector">LiPo Charger</text>
 <text x="5.08" y="104.14" size="3.81" layer="97" font="vector">Switching Regulator</text>
-<text x="169.418" y="7.112" size="2.1844" layer="94" font="vector">Marshall Taylor</text>
+<text x="166.878" y="11.43" size="2.1844" layer="94" font="vector">Marshall Taylor</text>
 <text x="238.76" y="7.62" size="2.54" layer="94" font="vector">vX2</text>
 <text x="132.08" y="139.7" size="1.778" layer="97" font="vector">500mA</text>
@@
 <text x="32.512" y="36.83" size="1.27" layer="97" font="vector">Install 100k resistor for
 inductor current limit</text>
-<text x="166.878" y="11.43" size="2.1844" layer="94" font="vector">Aaron Weiss/Patrick Alberts/Toni Klopfenstein</text>
 <text x="116.84" y="50.8" size="1.778" layer="97" font="vector">750k for 5v,
 450k (750k || 1.125k) for 3.3v</text>
@@
 <instance part="U$1" gate="G$1" x="134.62" y="10.16"/>
 <instance part="JP16" gate="G$1" x="246.38" y="20.32"/>
-<instance part="U$2" gate="G$1" x="148.844" y="7.366"/>
 <instance part="GND1" gate="1" x="210.82" y="149.86"/>
 <instance part="LOGO1" gate="G$1" x="116.84" y="2.54"/>
@@
 <instance part="JP4" gate="G$1" x="111.76" y="78.74" rot="R90"/>
 <instance part="J7" gate="G$1" x="213.36" y="134.62" rot="R180"/>
+<instance part="TP1" gate="G$1" x="101.6" y="170.18"/>
 </instances>
 <busses>
@@
 <pinref part="C3" gate="G$1" pin="1"/>
 <pinref part="JP1" gate="G$1" pin="2"/>
+<label x="53.34" y="78.74" size="1.27" layer="95"/>
 </segment>
 </net>
@@
 <pinref part="D4" gate="G$1" pin="C"/>
 <wire x1="96.52" y1="165.1" x2="99.06" y2="165.1" width="0.1524" layer="91"/>
+<pinref part="TP1" gate="G$1" pin="1"/>
+<wire x1="101.6" y1="170.18" x2="99.06" y2="170.18" width="0.1524" layer="91"/>
+<wire x1="99.06" y1="170.18" x2="99.06" y2="165.1" width="0.1524" layer="91"/>
+<junction x="99.06" y="165.1"/>
 </segment>
 </net>
@@
 <wire x1="172.72" y1="83.82" x2="172.72" y2="86.36" width="0.1524" layer="91"/>
 <junction x="172.72" y="86.36"/>
+<junction x="111.76" y="86.36"/>
 </segment>
 </net>
@@
 <wire x1="203.2" y1="152.4" x2="203.2" y2="134.62" width="0.1524" layer="91"/>
 <wire x1="203.2" y1="134.62" x2="205.74" y2="134.62" width="0.1524" layer="91"/>
-<junction x="200.66" y="152.4"/>
 <pinref part="J7" gate="G$1" pin="1"/>
+<junction x="203.2" y="152.4"/>
 </segment>
 </net>
@@
 </sheet>
 </sheets>
+<errors>
+</errors>
 </schematic>
 </drawing>
