File: Hardware/LiPoChargerBooster5V1A.brd (EAGLE design)
At the start: 20.3 x 31.8 mm, 38 parts, among them J1 AMP FCI 10103594-0001LF, J2 PTH, J3 PTH, J4 JST, J7 PTH, U1 MCP73831

Commit message: Ready for review
Parts:
- removed JP1: NC, SparkFun-Jumpers:SMT-JUMPER_2_NC_TRACE_NO-SILK
- removed JP4: JUMPER-SMT_2_NO_SILK, SparkFun-Jumpers:SMT-JUMPER_2_NO_SILK
- removed R7: 1.125M, SparkFun-Resistors:0603
- added R2: 10k, SparkFun-Resistors:0603
- L1: value 2.2µH/±20%/1.5A -> NEW2.2U; device DuplicatedCoils:INDUCTOR_2.2UHCOPY -> DuplicatedCoils:INDUCTOR_4X4MM
- U2: value SPARKFUN-POWERIC_PAM2401 -> PAM2401
- moved J6 19.1 mm to (7.62, 6.35)
- moved U$1 10.8 mm to (17.8, 29.2)
- moved JP3 2.45 mm to (19.2, 17.4)
- moved R6 1.71 mm to (12.4, 11.3)
- moved J2 0.90 mm to (7.62, 11.4)
- moved R1 0.76 mm to (13.8, 11.3)
- moved L1 0.76 mm to (16.4, 18.9), turned to 90 degrees
- moved C9 0.68 mm to (8.76, 13.7)
- renumbered U$3 to U2
Connections:
- removed net N$1: JP4.1, R7.2
- net EN: now also R2.1; no longer JP1.1
- net N$12: no longer R7.1
- net VBATT: now also R2.2; no longer JP1.2
- net VCC: no longer JP4.2
Routing:
- net VBATT: track 32.6 -> 46.7 mm
- net N$1: track 4.90 -> 0.00 mm, vias 1 -> 0
- net EN: track 12.6 -> 16.3 mm, vias 1 -> 2
- net N$2: track 5.73 -> 3.14 mm
- net VCC: track 21.2 -> 19.1 mm, vias 1 -> 0
- net N$12: track 6.48 -> 4.54 mm
- net GND: track 2.89 -> 3.78 mm, vias 15 -> 18
- net N$4: track 3.16 -> 3.79 mm
Other:
- board text added: "(Pulled up)"
- board text added: "5V OUT"
- board text added: "Charger Booster"
- board text added: "EN"
- board text added: "Max: 1A"
- board text added: "v10"
- board text removed: "ENB"
- board text removed: "LiPo Charge Boost"
- board text removed: "OUT"
- board text removed: "Open for 3.3v out"
- board text removed: "Open for ext. ENB"
- board text removed: "vX2"
