File: Hardware/LiPoChargerBooster5V1A.brd (EAGLE design)
At the start: 20.3 x 31.8 mm, 36 parts, among them J1 AMP FCI 10103594-0001LF, J2 PTH, J3 PTH, J4 JST, J7 PTH, U1 MCP73831, U2 PAM2401

Commit message: Post reivew changes
Parts:
- added JP1, JP4: FIDUCIAL1X2, SparkFun-Aesthetics:FIDUCIAL-1X2
- moved JP16 6.14 mm to (10.0, 30.7)
Other:
- board text removed: "(Pulled up)"
Changed lines of the file:
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@@
 <layer number="37" name="tTest" color="7" fill="1" visible="no" active="yes"/>
 <layer number="38" name="bTest" color="7" fill="1" visible="no" active="yes"/>
-<layer number="39" name="tKeepout" color="4" fill="11" visible="yes" active="yes"/>
-<layer number="40" name="bKeepout" color="1" fill="11" visible="yes" active="yes"/>
+<layer number="39" name="tKeepout" color="4" fill="11" visible="no" active="yes"/>
+<layer number="40" name="bKeepout" color="1" fill="11" visible="no" active="yes"/>
 <layer number="41" name="tRestrict" color="4" fill="10" visible="no" active="yes"/>
 <layer number="42" name="bRestrict" color="1" fill="10" visible="no" active="yes"/>
@@
 <wire x1="20.32" y1="31.75" x2="0" y2="31.75" width="0.2032" layer="20"/>
 <wire x1="0" y1="31.75" x2="0" y2="0" width="0.2032" layer="20"/>
-<text x="3.7671375" y="10.652125" size="0.8128" layer="22" font="vector" ratio="18" rot="MR270">(Pulled up)</text>
 <text x="12.446" y="22.987" size="1.27" layer="21" font="vector" ratio="18" align="top-left">-</text>
 <text x="18.415" y="22.987" size="1.27" layer="21" font="vector" ratio="18" rot="R180">+</text>
@@
 <text x="18.8515625" y="2.5193625" size="0.8128" layer="22" font="vector" ratio="18" rot="MR0">Max: 1A</text>
 <text x="9.1201875" y="5.762625" size="0.8128" layer="22" font="vector" ratio="18" rot="MR90">EN</text>
-<wire x1="6.588125" y1="5.476875" x2="6.3103125" y2="5.1990625" width="0.2032" layer="22"/>
-<wire x1="6.3103125" y1="5.1990625" x2="4.206875" y2="5.1990625" width="0.2032" layer="22"/>
 </plain>
 <attributes>
@@
 <element name="JP7" library="SparkFun" package="STAND-OFF" value="STAND-OFF" x="6.35" y="29.21"/>
 <element name="U$1" library="SparkFun" package="OSHW-LOGO-S" value="OSHW-LOGOS" x="17.78" y="29.21" rot="MR0"/>
-<element name="JP16" library="SparkFun-Aesthetics" package="FIDUCIAL-1X2" value="FIDUCIAL1X2" x="16.129" y="30.099"/>
+<element name="JP16" library="SparkFun-Aesthetics" package="FIDUCIAL-1X2" value="FIDUCIAL1X2" x="10.017125" y="30.654625"/>
 <element name="FRAME1" library="SparkFun-Aesthetics" package="CREATIVE_COMMONS" value="FRAME-LETTER" x="-24.4323125" y="-24.4475" smashed="yes"/>
 <element name="LOGO1" library="SparkFun-Aesthetics" package="SFE_LOGO_FLAME_.1" value="SFE_LOGO_FLAME.1_INCH" x="0.762" y="0.508"/>
@@
 </element>
 <element name="L1" library="DuplicatedCoils" package="INDUCTOR_4X4MM" value="NEW2.2U" x="16.383" y="18.923" rot="R90"/>
+<element name="JP1" library="SparkFun-Aesthetics" package="FIDUCIAL-1X2" value="FIDUCIAL1X2" x="3.81" y="30.48" rot="MR0"/>
+<element name="JP4" library="SparkFun-Aesthetics" package="FIDUCIAL-1X2" value="FIDUCIAL1X2" x="13.0175" y="1.905" rot="MR0"/>
 </elements>
 <signals>
@@
 <wire x1="6.92358125" y1="8.19358125" x2="7.62" y2="8.89" width="0.4064" layer="1"/>
 <via x="8.763" y="10.16" extent="1-16" drill="0.381"/>
-<via x="8.89" y="1.27" extent="1-16" drill="0.381"/>
+<via x="9.286875" y="0.9525" extent="1-16" drill="0.381"/>
 <via x="19.431" y="2.54" extent="1-16" drill="0.381"/>
 <via x="19.431" y="6.096" extent="1-16" drill="0.381"/>
@@
 <via x="7.62" y="24.13" extent="1-16" drill="0.381"/>
 <via x="10.16" y="24.13" extent="1-16" drill="0.381"/>
-<via x="9.525" y="30.48" extent="1-16" drill="0.381"/>
-<via x="3.175" y="30.48" extent="1-16" drill="0.381"/>
+<via x="9.525" y="29.21" extent="1-16" drill="0.381"/>
+<via x="3.175" y="29.21" extent="1-16" drill="0.381"/>
 <via x="2.413" y="17.145" extent="1-16" drill="0.381"/>
 <via x="15.367" y="12.954" extent="1-16" drill="0.381"/>
 <via x="11.303" y="11.303" extent="1-16" drill="0.381"/>
-<via x="10.16" y="3.81" extent="1-16" drill="0.381"/>
+<via x="11.43" y="2.8575" extent="1-16" drill="0.381"/>
 </signal>
 <signal name="5VIN">
@@
 <wire x1="1.27" y1="21.463" x2="2.413" y2="20.32" width="0.8128" layer="16"/>
 <wire x1="2.413" y1="20.32" x2="2.54" y2="20.32" width="0.8128" layer="16"/>
-<wire x1="2.54" y1="20.32" x2="5.08" y2="20.32" width="0.8128" layer="16"/>
+<wire x1="2.54" y1="20.32" x2="3.81" y2="20.32" width="0.8128" layer="16"/>
+<wire x1="3.81" y1="20.32" x2="5.08" y2="20.32" width="0.8128" layer="16"/>
 <wire x1="5.08" y1="20.32" x2="5.207" y2="20.32" width="0.8128" layer="16"/>
 <via x="5.08" y="20.32" extent="1-16" drill="0.508"/>
@@
 <wire x1="14.843125" y1="19.9628125" x2="14.843125" y2="18.989675" width="0.8128" layer="1"/>
 <wire x1="14.843125" y1="18.989675" x2="14.9098" y2="18.923" width="0.8128" layer="1"/>
-<wire x1="5.08" y1="20.32" x2="3.81" y2="20.32" width="0" layer="19" extent="1-1"/>
 </signal>
 <signal name="N$11">

Commit message: Updated components and checked against the checklist, moved temp parts into normal eagle libs
Parts:
- L1: value NEW2.2U -> 2.2UH3A; device DuplicatedCoils:INDUCTOR_4X4MM -> SparkFun-Coils:INDUCTOR_4X4MM
- U2: device Apo Board 2017 ATmega328SMD_PAM2401:SPARKFUN-POWERIC_MSOP8 -> SparkFun-IC-Power:MSOP8
Other:
- board text added: "5V, 1A"
- board text added: "OUT"
- board text removed: "5V OUT"
- board text removed: "Max: 1A"
