File: Hardware/LiPoChargerBooster5V1A.brd (EAGLE design)
At the start: 20.3 x 31.8 mm, 38 parts, among them J1 AMP FCI 10103594-0001LF, J2 PTH, J3 PTH, J4 JST, J7 PTH, U1 MCP73831, U2 PAM2401

Commit message: Changed pull up to 750k, added photos
Parts:
- R2: value 10k -> 750K
Changed lines of the file:
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@@
 <element name="J7" library="SparkFun-Connectors" package="1X02" value="PTH" x="1.27" y="27.94" rot="R270"/>
 <element name="TP1" library="SparkFun-Connectors" package="PAD.03X.03" value="TEST-POINT3" x="4.064" y="16.51" rot="MR0"/>
-<element name="R2" library="SparkFun-Resistors" package="0603" value="10k" x="10.16" y="11.303" rot="R90">
-<attribute name="PROD_ID" value="RES-00824" x="10.16" y="11.303" size="1.778" layer="27" rot="R90" display="off"/>
+<element name="R2" library="SparkFun-Resistors" package="0603" value="750K" x="10.16" y="11.303" rot="R90">
+<attribute name="PROD_ID" value="RES-13768" x="10.16" y="11.303" size="1.778" layer="27" rot="R90" display="off"/>
 </element>
 <element name="L1" library="SparkFun-Coils" package="INDUCTOR_4X4MM" value="2.2UH3A" x="16.383" y="18.923" rot="R90">
