File: Hardware/LiPoChargerBooster5V1A.sch (EAGLE design)
At the start: 38 parts, among them J1 AMP FCI 10103594-0001LF, J2 PTH, J3 PTH, J4 JST, J7 PTH, U1 MCP73831

Commit message: Ready for review
Parts:
- removed JP1: NC, SparkFun-Jumpers:JUMPER-SMT_2_NC_TRACE_NO-SILK
- removed JP4: JUMPER-SMT_2_NO_SILK, SparkFun-Jumpers:JUMPER-SMT_2_NO_SILK
- removed R7: 1.125M, SparkFun-Resistors:750OHM-0603-1/10W-1%
- added R2: 10k, SparkFun-Resistors:10KOHM-0603-1/10W-1%
- L1: value 2.2µH/±20%/1.5A -> NEW2.2U; device DuplicatedCoils:INDUCTORCOPY-VLF4012AT-2.2UH -> DuplicatedCoils:NEW2.2U
- U2: value SPARKFUN-POWERIC_PAM2401 -> PAM2401
- renumbered U$3 to U2
Connections:
- removed net N$1: JP4.1, R7.2
- net EN: now also R2.1; no longer JP1.1
- net N$12: no longer R7.1
- net VBATT: now also R2.2; no longer JP1.2
- net VCC: no longer JP4.2
Other:
- note added: "0.9V-to-5V Step Up PAM2401 1A capacity available above 3.0V"
- note added: "v10"
- note removed: "0.9V-to-5V Step Up PAM2401"
- note removed: "750k for 5v, 450k (750k || 1.125k) for 3.3v"
- note removed: "ATMEGA328P-AU"
- note removed: "vX2"
Changed lines of the file:
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@@
 <part name="GND24" library="SparkFun" deviceset="GND" device=""/>
 <part name="GND5" library="SparkFun" deviceset="GND" device=""/>
-<part name="U$3" library="Apo Board 2017 ATmega328SMD_PAM2401" deviceset="SPARKFUN-POWERIC_PAM2401" device=""/>
-<part name="L1" library="DuplicatedCoils" deviceset="INDUCTORCOPY" device="-VLF4012AT-2.2UH" value="2.2µH/±20%/1.5A"/>
+<part name="U2" library="Apo Board 2017 ATmega328SMD_PAM2401" deviceset="SPARKFUN-POWERIC_PAM2401" device="" value="PAM2401"/>
 <part name="J2" library="SparkFun-Connectors" deviceset="CONN_02" device="" value="PTH"/>
 <part name="J3" library="SparkFun-Connectors" deviceset="CONN_02" device="" value="PTH"/>
@@
 <part name="C2" library="SparkFun-Capacitors" deviceset="22UF" device="-0805-6.3V-20%" value="22uF"/>
 <part name="C3" library="SparkFun-Capacitors" deviceset="22UF" device="-0805-6.3V-20%" value="22uF"/>
-<part name="JP1" library="SparkFun-Jumpers" deviceset="JUMPER-SMT_2_NC_TRACE" device="_NO-SILK" value="NC"/>
 <part name="J5" library="SparkFun-Connectors" deviceset="CONN_02" device=""/>
 <part name="J6" library="SparkFun-Connectors" deviceset="CONN_01" device=""/>
@@
 <part name="J1" library="SparkFun-Connectors" deviceset="USB_MICRO-B" device="_HALF_PTH" value="AMP FCI 10103594-0001LF"/>
 <part name="S2" library="SparkFun-Switches" deviceset="SWITCH-DPDT" device="-SMD-AYZ0202"/>
-<part name="R7" library="SparkFun-Resistors" deviceset="750OHM" device="-0603-1/10W-1%" value="1.125M"/>
-<part name="JP4" library="SparkFun-Jumpers" deviceset="JUMPER-SMT_2_NO" device="_SILK"/>
 <part name="J7" library="SparkFun-Connectors" deviceset="CONN_02" device="" value="PTH"/>
 <part name="TP1" library="SparkFun-Connectors" deviceset="TEST-POINT" device="3"/>
+<part name="R2" library="SparkFun-Resistors" deviceset="10KOHM" device="-0603-1/10W-1%" value="10k"/>
+<part name="L1" library="DuplicatedCoils" deviceset="NEW2.2U" device=""/>
 </parts>
 <sheets>
@@
 <text x="5.08" y="104.14" size="3.81" layer="97" font="vector">Switching Regulator</text>
 <text x="166.878" y="11.43" size="2.1844" layer="94" font="vector">Marshall Taylor</text>
-<text x="238.76" y="7.62" size="2.54" layer="94" font="vector">vX2</text>
+<text x="238.76" y="7.62" size="2.54" layer="94" font="vector">v10</text>
 <text x="132.08" y="139.7" size="1.778" layer="97" font="vector">500mA</text>
 <text x="137.16" y="127" size="1.778" layer="97" font="vector">Ireg = 1000V/Rprog</text>
-<text x="63.5" y="86.36" size="2.54" layer="97" font="vector">0.9V-to-5V Step Up
-PAM2401 </text>
-<text x="66.04" y="33.02" size="2.54" layer="97" font="vector">ATMEGA328P-AU</text>
+<text x="5.08" y="91.44" size="2.54" layer="97" font="vector">0.9V-to-5V Step Up
+PAM2401
+1A capacity available above 3.0V</text>
 <text x="32.512" y="36.83" size="1.27" layer="97" font="vector">Install 100k resistor for
 inductor current limit</text>
-<text x="116.84" y="50.8" size="1.778" layer="97" font="vector">750k for 5v,
-450k (750k || 1.125k) for 3.3v</text>
 <text x="205.74" y="124.46" size="1.778" layer="97" font="vector">Switch Bypass</text>
 </plain>
@@
 <instance part="GND17" gate="1" x="149.86" y="134.62"/>
 <instance part="JP3" gate="G$1" x="190.5" y="33.02"/>
-<instance part="JP6" gate="G$1" x="241.3" y="33.02"/>
-<instance part="JP7" gate="G$1" x="241.3" y="27.94"/>
+<instance part="JP6" gate="G$1" x="241.3" y="27.94"/>
+<instance part="JP7" gate="G$1" x="233.68" y="27.94"/>
 <instance part="GND6" gate="1" x="208.28" y="66.04"/>
 <instance part="P+1" gate="G$1" x="182.88" y="96.52"/>
 <instance part="U$1" gate="G$1" x="134.62" y="10.16"/>
-<instance part="JP16" gate="G$1" x="246.38" y="20.32"/>
+<instance part="JP16" gate="G$1" x="226.06" y="27.94"/>
 <instance part="GND1" gate="1" x="210.82" y="149.86"/>
 <instance part="LOGO1" gate="G$1" x="116.84" y="2.54"/>
@@
 <instance part="GND24" gate="1" x="160.02" y="68.58" rot="MR0"/>
 <instance part="GND5" gate="1" x="172.72" y="58.42" rot="MR0"/>
-<instance part="U$3" gate="G$1" x="76.2" y="60.96"/>
-<instance part="L1" gate="G$1" x="76.2" y="78.74" rot="R90"/>
+<instance part="U2" gate="G$1" x="76.2" y="60.96" smashed="yes">
+<attribute name="NAME" x="71.12" y="75.184" size="1.778" layer="95"/>
+<attribute name="VALUE" x="68.834" y="44.958" size="1.778" layer="96"/>
+</instance>
 <instance part="J2" gate="G$1" x="53.34" y="167.64"/>
 <instance part="J3" gate="G$1" x="220.98" y="172.72" rot="R180"/>
@@
 <instance part="C2" gate="G$1" x="149.86" y="76.2"/>
 <instance part="C3" gate="G$1" x="50.8" y="71.12"/>
-<instance part="JP1" gate="G$1" x="60.96" y="63.5" rot="R90"/>
 <instance part="J5" gate="G$1" x="218.44" y="81.28" rot="R180"/>
 <instance part="J6" gate="G$1" x="40.64" y="55.88"/>
-<instance part="JP2" gate="G$1" x="241.3" y="20.32"/>
+<instance part="JP2" gate="G$1" x="218.44" y="27.94"/>
 <instance part="J1" gate="G$1" x="55.88" y="152.4" rot="MR0"/>
 <instance part="S2" gate="G$1" x="195.58" y="154.94"/>
-<instance part="R7" gate="G$1" x="111.76" y="66.04" rot="R90"/>
-<instance part="JP4" gate="G$1" x="111.76" y="78.74" rot="R90"/>
 <instance part="J7" gate="G$1" x="213.36" y="134.62" rot="R180"/>
 <instance part="TP1" gate="G$1" x="101.6" y="170.18"/>
+<instance part="R2" gate="G$1" x="60.96" y="63.5" rot="R90"/>
+<instance part="L1" gate="G$1" x="76.2" y="78.74" rot="R90"/>
 </instances>
 <busses>
@@
 <wire x1="88.9" y1="50.8" x2="91.44" y2="50.8" width="0.1524" layer="91"/>
 <junction x="91.44" y="50.8"/>
-<pinref part="U$3" gate="G$1" pin="AGND"/>
-<pinref part="U$3" gate="G$1" pin="PGND"/>
+<pinref part="U2" gate="G$1" pin="AGND"/>
+<pinref part="U2" gate="G$1" pin="PGND"/>
 </segment>
 <segment>
@@
 <wire x1="50.8" y1="76.2" x2="50.8" y2="78.74" width="0.1524" layer="91"/>
 <wire x1="60.96" y1="71.12" x2="60.96" y2="78.74" width="0.1524" layer="91"/>
+<pinref part="U2" gate="G$1" pin="VIN"/>
+<pinref part="C3" gate="G$1" pin="1"/>
+<label x="53.34" y="78.74" size="1.27" layer="95"/>
+<pinref part="R2" gate="G$1" pin="2"/>
 <wire x1="60.96" y1="68.58" x2="60.96" y2="71.12" width="0.1524" layer="91"/>
 <junction x="60.96" y="71.12"/>
-<pinref part="U$3" gate="G$1" pin="VIN"/>
 <pinref part="L1" gate="G$1" pin="1"/>
-<pinref part="C3" gate="G$1" pin="1"/>
-<pinref part="JP1" gate="G$1" pin="2"/>
-<label x="53.34" y="78.74" size="1.27" layer="95"/>
 </segment>
 </net>
@@
 <pinref part="R4" gate="G$1" pin="2"/>
 <wire x1="99.06" y1="86.36" x2="99.06" y2="78.74" width="0.1524" layer="91"/>
-<wire x1="99.06" y1="86.36" x2="111.76" y2="86.36" width="0.1524" layer="91"/>
 <junction x="99.06" y="86.36"/>
-<wire x1="111.76" y1="86.36" x2="149.86" y2="86.36" width="0.1524" layer="91"/>
+<wire x1="99.06" y1="86.36" x2="149.86" y2="86.36" width="0.1524" layer="91"/>
 <wire x1="149.86" y1="86.36" x2="149.86" y2="81.28" width="0.1524" layer="91"/>
 <junction x="149.86" y="86.36"/>
@@
 <junction x="200.66" y="81.28"/>
 <junction x="195.58" y="81.28"/>
-<pinref part="U$3" gate="G$1" pin="OUT"/>
+<pinref part="U2" gate="G$1" pin="OUT"/>
 <pinref part="D1" gate="G$1" pin="C"/>
 <pinref part="D2" gate="G$1" pin="C"/>
@@
 <pinref part="C2" gate="G$1" pin="1"/>
 <pinref part="J5" gate="G$1" pin="1"/>
-<pinref part="JP4" gate="G$1" pin="2"/>
-<wire x1="111.76" y1="86.36" x2="111.76" y2="83.82" width="0.1524" layer="91"/>
 <pinref part="D3" gate="G$1" pin="A"/>
 <wire x1="172.72" y1="83.82" x2="172.72" y2="86.36" width="0.1524" layer="91"/>
 <junction x="172.72" y="86.36"/>
-<junction x="111.76" y="86.36"/>
 </segment>
 </net>
@@
 <segment>
 <wire x1="48.26" y1="55.88" x2="60.96" y2="55.88" width="0.1524" layer="91"/>
-<wire x1="60.96" y1="55.88" x2="60.96" y2="58.42" width="0.1524" layer="91"/>
 <label x="53.34" y="55.88" size="1.778" layer="95" font="vector" rot="MR0"/>
-<wire x1="63.5" y1="55.88" x2="60.96" y2="55.88" width="0.1524" layer="91"/>
+<pinref part="U2" gate="G$1" pin="EN"/>
+<pinref part="J6" gate="G$1" pin="1"/>
+<pinref part="R2" gate="G$1" pin="1"/>
+<wire x1="60.96" y1="55.88" x2="63.5" y2="55.88" width="0.1524" layer="91"/>
+<wire x1="60.96" y1="58.42" x2="60.96" y2="55.88" width="0.1524" layer="91"/>
 <junction x="60.96" y="55.88"/>
-<pinref part="U$3" gate="G$1" pin="EN"/>
-<pinref part="JP1" gate="G$1" pin="1"/>
-<pinref part="J6" gate="G$1" pin="1"/>
 </segment>
 </net>
@@
 <wire x1="99.06" y1="53.34" x2="99.06" y2="58.42" width="0.1524" layer="91"/>
 <wire x1="99.06" y1="60.96" x2="99.06" y2="58.42" width="0.1524" layer="91"/>
-<pinref part="U$3" gate="G$1" pin="FB"/>
+<pinref part="U2" gate="G$1" pin="FB"/>
 <junction x="99.06" y="60.96"/>
-<pinref part="R7" gate="G$1" pin="1"/>
 <wire x1="99.06" y1="58.42" x2="99.06" y2="68.58" width="0.1524" layer="91"/>
-<wire x1="111.76" y1="60.96" x2="111.76" y2="58.42" width="0.1524" layer="91"/>
-<wire x1="111.76" y1="58.42" x2="99.06" y2="58.42" width="0.1524" layer="91"/>
 <junction x="99.06" y="58.42"/>
 </segment>
@@
 <wire x1="91.44" y1="78.74" x2="91.44" y2="71.12" width="0.1524" layer="91"/>
 <wire x1="91.44" y1="71.12" x2="88.9" y2="71.12" width="0.1524" layer="91"/>
-<pinref part="U$3" gate="G$1" pin="LX"/>
+<pinref part="U2" gate="G$1" pin="LX"/>
 <pinref part="L1" gate="G$1" pin="2"/>
 </segment>
@@
 <wire x1="63.5" y1="50.8" x2="60.96" y2="50.8" width="0.1524" layer="91"/>
 <wire x1="60.96" y1="50.8" x2="60.96" y2="48.26" width="0.1524" layer="91"/>
-<pinref part="U$3" gate="G$1" pin="RSET"/>
+<pinref part="U2" gate="G$1" pin="RSET"/>
 </segment>
 </net>
@@
 </segment>
 </net>
-<net name="N$1" class="0">
-<segment>
-<pinref part="JP4" gate="G$1" pin="1"/>
-<pinref part="R7" gate="G$1" pin="2"/>
-<wire x1="111.76" y1="73.66" x2="111.76" y2="71.12" width="0.1524" layer="91"/>
-</segment>
-</net>

Commit message: Post reivew changes
Parts:
- added JP1, JP4: FIDUCIAL1X2, SparkFun-Aesthetics:FIDUCIAL1X2
Other:
- note added: "2.0K resistor placed for 500mA charge rate"
- note added: "Battery connection"
- note added: "Charge power"
- note added: "Charger"
- note added: "Enable"
- note added: "Enable pin: To disable output, short EN pin to ground (is pulled up with 10kOhm)"
- note added: "For heavy duty use: Use 2A switch in switch bypass pins, or jump with wire."
- note added: "LiPo Charger Booster"
- note added: "Output capacity: 5V, 1A for 3.0V to 4.2V battery voltage."
- note added: "Switch bypass"
- note added: "To charge battery, Minimize output load (or disable) Supply 3.75 to 6V, 500mA capable to USB or input voltage pins."
- note removed: "0.9V-to-5V Step Up PAM2401 1A capacity available above 3.0V"
- note removed: "500mA"
- note removed: "LiPo Charger"
- note removed: "Switch Bypass"
- moved on the sheet: C1, C10, C2, C3, C9, D1, D2, D3, D4, J1, J2, J3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

Commit message: Updated components and checked against the checklist, moved temp parts into normal eagle libs
Parts:
- L1: value NEW2.2U -> 2.2UH3A; device DuplicatedCoils:NEW2.2U -> SparkFun-Coils:INDUCTOR-IFSC1515AHER2R2M01
- R4: device SparkFun-Resistors:750OHM-0603-1/10W-1% -> SparkFun-Resistors:750KOHM-0603-1/10W-1%
- U2: device Apo Board 2017 ATmega328SMD_PAM2401:SPARKFUN-POWERIC_PAM2401 -> SparkFun-IC-Power:PAM2401
Changed lines of the file:
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@@
 <part name="U1" library="SparkFun-IC-Power" deviceset="MCP73831" device=""/>
 <part name="GND2" library="SparkFun" deviceset="GND" device=""/>
-<part name="R4" library="SparkFun-Resistors" deviceset="750OHM" device="-0603-1/10W-1%" value="750K"/>
+<part name="R4" library="SparkFun-Resistors" deviceset="750KOHM" device="-0603-1/10W-1%" value="750K"/>
 <part name="R1" library="SparkFun-Resistors" deviceset="100KOHM" device="-0603-1/10W-1%" value="100k"/>
 <part name="GND3" library="SparkFun" deviceset="GND" device=""/>
@@
 <part name="GND24" library="SparkFun" deviceset="GND" device=""/>
 <part name="GND5" library="SparkFun" deviceset="GND" device=""/>
-<part name="U2" library="Apo Board 2017 ATmega328SMD_PAM2401" deviceset="SPARKFUN-POWERIC_PAM2401" device="" value="PAM2401"/>
+<part name="U2" library="SparkFun-IC-Power" deviceset="PAM2401" device="" value="PAM2401"/>
 <part name="J2" library="SparkFun-Connectors" deviceset="CONN_02" device="" value="PTH"/>
 <part name="J3" library="SparkFun-Connectors" deviceset="CONN_02" device="" value="PTH"/>
@@
 <part name="TP1" library="SparkFun-Connectors" deviceset="TEST-POINT" device="3"/>
 <part name="R2" library="SparkFun-Resistors" deviceset="10KOHM" device="-0603-1/10W-1%" value="10k"/>
-<part name="L1" library="DuplicatedCoils" deviceset="NEW2.2U" device=""/>
+<part name="L1" library="SparkFun-Coils" deviceset="INDUCTOR" device="-IFSC1515AHER2R2M01" value="2.2UH3A"/>
 <part name="JP1" library="SparkFun-Aesthetics" deviceset="FIDUCIAL" device="1X2"/>
 <part name="JP4" library="SparkFun-Aesthetics" deviceset="FIDUCIAL" device="1X2"/>
@@
 <segment>
 <wire x1="182.88" y1="144.78" x2="182.88" y2="147.32" width="0.1524" layer="91"/>
-<wire x1="154.94" y1="147.32" x2="182.88" y2="147.32" width="0.1524" layer="91"/>
-<label x="184.912" y="147.574" size="1.778" layer="95" font="vector"/>
+<wire x1="154.94" y1="147.32" x2="175.26" y2="147.32" width="0.1524" layer="91"/>
+<label x="175.26" y="149.86" size="1.27" layer="95" font="vector" rot="R90" xref="yes"/>
 <pinref part="C10" gate="G$1" pin="1"/>
 <pinref part="U1" gate="G$1" pin="VBAT"/>
 <junction x="182.88" y="147.32"/>
+<wire x1="175.26" y1="147.32" x2="182.88" y2="147.32" width="0.1524" layer="91"/>
 <wire x1="195.58" y1="147.32" x2="193.04" y2="147.32" width="0.1524" layer="91"/>
 <pinref part="S2" gate="G$1" pin="2"/>
@@
 <junction x="193.04" y="139.7"/>
 <pinref part="J7" gate="G$1" pin="2"/>
+<wire x1="175.26" y1="147.32" x2="175.26" y2="149.86" width="0.1524" layer="91"/>
+<junction x="175.26" y="147.32"/>
 </segment>
 <segment>
@@
 <pinref part="U2" gate="G$1" pin="VIN"/>
 <pinref part="C3" gate="G$1" pin="1"/>
-<label x="58.42" y="63.5" size="1.27" layer="95"/>
+<label x="55.88" y="66.04" size="1.27" layer="95" rot="R90" xref="yes"/>
 <pinref part="R2" gate="G$1" pin="2"/>
 <wire x1="66.04" y1="53.34" x2="66.04" y2="55.88" width="0.1524" layer="91"/>
 <junction x="66.04" y="55.88"/>
 <pinref part="L1" gate="G$1" pin="1"/>
+<junction x="55.88" y="63.5"/>
+<wire x1="55.88" y1="63.5" x2="55.88" y2="66.04" width="0.1524" layer="91"/>
 </segment>
 </net>

Commit message: Changed pull up to 750k, added photos
Parts:
- R2: value 10k -> 750K; device SparkFun-Resistors:10KOHM-0603-1/10W-1% -> SparkFun-Resistors:750KOHM-0603-1/10W-1%
Changed lines of the file:
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@@
 <part name="J7" library="SparkFun-Connectors" deviceset="CONN_02" device="" value="PTH"/>
 <part name="TP1" library="SparkFun-Connectors" deviceset="TEST-POINT" device="3"/>
-<part name="R2" library="SparkFun-Resistors" deviceset="10KOHM" device="-0603-1/10W-1%" value="10k"/>
+<part name="R2" library="SparkFun-Resistors" deviceset="750KOHM" device="-0603-1/10W-1%" value="750K"/>
 <part name="L1" library="SparkFun-Coils" deviceset="INDUCTOR" device="-IFSC1515AHER2R2M01" value="2.2UH3A"/>
 <part name="JP1" library="SparkFun-Aesthetics" deviceset="FIDUCIAL" device="1X2"/>
